File: imuDevBoard.kicad_pcb (KiCad board)
At the start: 2 copper layers, 39 parts, among them J1 USB_C_Receptacle_USB2.0_16P, SW1 SW_Push, SW2 SW_SPDT, U1 RP2350A, U2 W25Q128JVS, U3 TLV75533PDBV, U4 ICM-42688-P, Y1 Crystal_GND24, 12MHz

Commit message: fixed design
Parts:
- moved C22 2.62 mm to (74.2, 107.0)
- moved C7 1.44 mm to (70.5, 110.0)
- moved Y1 0.71 mm to (71.6, 107.3)
- moved U4 0.59 mm to (76.4, 106.0), turned to 90 degrees
- moved R8 0.58 mm to (74.3, 102.0), turned to 0 degrees
- moved C1 0.28 mm to (64.0, 109.5)
- moved C17 0.28 mm to (65.5, 110.0)
- moved U3 0.28 mm to (65.9, 107.0)
- moved D1 0.07 mm to (76.0, 102.7)
- moved C2 0.05 mm to (78.0, 102.7)
Routing:
- net GND: track 0.00 -> 96.0 mm, vias 0 -> 14
- net +3V3: track 49.3 -> 86.4 mm, vias 0 -> 10
- net (no net): track 13.0 -> 0.00 mm, vias 2 -> 0
- net Net-(U1-~{QSPI_SS}): track 11.0 -> 23.9 mm, vias 2 -> 3
- net Net-(U1-XIN): track 2.75 -> 14.6 mm
- net Net-(U1-QSPI_SCLK): track 1.15 -> 12.2 mm, vias 1 -> 2
- net Net-(U1-VREG_FB): track 16.0 -> 26.9 mm
- net Net-(U1-GPIO17): track 0.00 -> 10.8 mm, vias 0 -> 2
- net Net-(U1-GPIO20): track 0.00 -> 10.3 mm, vias 0 -> 2
- net Net-(U1-GPIO18): track 0.00 -> 8.86 mm, vias 0 -> 2
- net Net-(U1-GPIO16): track 0.00 -> 8.57 mm, vias 0 -> 2
- net Net-(U1-GPIO21): track 0.00 -> 8.28 mm, vias 0 -> 2
- net Net-(U1-GPIO19): track 0.00 -> 5.26 mm, vias 0 -> 2
- net Net-(U1-GPIO25): track 0.00 -> 3.50 mm, vias 0 -> 2
- net Net-(U1-QSPI_SD3): track 6.55 -> 9.09 mm
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Other:
- board outline added: 33 x 26 mm

Commit message: fixed all errors on pcb
Routing:
- net GND: track 96.0 -> 107.8 mm, vias 14 -> 16
- net Net-(U1-VREG_LX): track 4.64 -> 8.75 mm, vias 0 -> 2
- net +3V3: track 86.4 -> 88.5 mm, vias 10 -> 9
- net Net-(U1-VREG_FB): track 26.9 -> 26.2 mm
